File: board_v11/RGB_Station_v11.sch (EAGLE design)
At the start: 44 parts, among them IC1 MCP1702T-3302E/MB, J1 M20, J2 M20, J3 USB_MICRO, U1 PIC32MX270F256D_44VTLA_44, U2 74LVC2T45, U3 MCP121T-315E/TT, U4 DSC6111CI1A-008.0000, U6 RN4871

Commit message: Updated switches with proper footprint.
Parts:
- removed S1, S2: SWITCH-MOMENTARY-SPSTSMD-3, SparkFun-Retired:SWITCH-MOMENTARY-SPSTSMD-3
- added SW1, SW2: KMR2_SWITCH, kmr2_switch:KMR2_SWITCH
Connections:
- net !MCLR!: now also SW2.P3, SW2.P4; no longer S2.2
- net GND: now also SW1.P1, SW1.P2, SW2.P1, SW2.P2; no longer S1.1, S2.1
- net RA8: now also SW1.P3, SW1.P4; no longer S1.2

Commit message: Routed new switches, tweaked layout a bit - blue LED now on very end.
Parts:
- R11, R4, R8: value 1K -> 8.2K
Connections:
- removed net N$10: LED3.A, R4.1
- removed net N$9: LED3.C, U6.P0_2
- new net N$1: R4.2, U6.P0_2
- new net N$5: LED3.C, R4.1
- net 3.3V: now also LED3.A; no longer R4.2
Other:
- moved on the sheet: LED3, R4
Changed lines of the file:
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@@
 <?xml version="1.0" encoding="utf-8"?>
 <!DOCTYPE eagle SYSTEM "eagle.dtd">
-<eagle version="6.6.0">
+<eagle version="7.7.0">
 <drawing>
 <settings>
@@
 <part name="GND5" library="SparkFun02-20-08" deviceset="GND" device=""/>
 <part name="P+4" library="SparkFun02-20-08" deviceset="3.3V" device=""/>
-<part name="R8" library="SparkFun" deviceset="RESISTOR" device="0603-RES" value="1K"/>
+<part name="R8" library="SparkFun" deviceset="RESISTOR" device="0603-RES" value="8.2K"/>
 <part name="LED2" library="SparkFun" deviceset="LED" device="0603" value="GREEN"/>
 <part name="GND19" library="SparkFun02-20-08" deviceset="GND" device=""/>
@@
 <part name="R9" library="SparkFun" deviceset="RESISTOR" device="0603-RES" value="10K"/>
 <part name="R10" library="SparkFun" deviceset="RESISTOR" device="0603-RES" value="10K"/>
-<part name="R11" library="SparkFun" deviceset="RESISTOR" device="0603-RES" value="1K"/>
+<part name="R11" library="SparkFun" deviceset="RESISTOR" device="0603-RES" value="8.2K"/>
 <part name="LED1" library="SparkFun" deviceset="LED" device="0603" value="RED"/>
 <part name="GND4" library="SparkFun02-20-08" deviceset="GND" device=""/>
@@
 <part name="GND15" library="SparkFun02-20-08" deviceset="GND" device=""/>
 <part name="VIN_5V" library="SparkFun02-20-08" deviceset="5V" device="" value="5V"/>
-<part name="R4" library="SparkFun" deviceset="RESISTOR" device="0603-RES" value="1K"/>
+<part name="R4" library="SparkFun" deviceset="RESISTOR" device="0603-RES" value="8.2K"/>
 <part name="LED3" library="SparkFun" deviceset="LED" device="0603" value="Blue"/>
 <part name="P+9" library="SparkFun02-20-08" deviceset="3.3V" device=""/>
@@
 <attribute name="VALUE" x="57.404" y="69.342" size="1.27" layer="96" font="vector"/>
 </instance>
-<instance part="R4" gate="G$1" x="337.82" y="137.16" smashed="yes" rot="R90">
-<attribute name="NAME" x="339.598" y="138.1506" size="1.27" layer="95" font="vector"/>
-<attribute name="VALUE" x="339.598" y="135.382" size="1.27" layer="96" font="vector"/>
-</instance>
-<instance part="LED3" gate="G$1" x="332.74" y="129.54" smashed="yes" rot="R270">
-<attribute name="NAME" x="325.374" y="127.762" size="1.27" layer="95" font="vector"/>
-<attribute name="VALUE" x="333.248" y="127.889" size="1.27" layer="96" font="vector"/>
+<instance part="R4" gate="G$1" x="330.2" y="129.54" smashed="yes" rot="R180">
+<attribute name="NAME" x="327.152" y="126.7206" size="1.27" layer="95" font="vector"/>
+<attribute name="VALUE" x="331.47" y="126.746" size="1.27" layer="96" font="vector"/>
+</instance>
+<instance part="LED3" gate="G$1" x="337.82" y="137.16" smashed="yes">
+<attribute name="NAME" x="331.47" y="136.652" size="1.27" layer="95" font="vector"/>
+<attribute name="VALUE" x="332.486" y="132.207" size="1.27" layer="96" font="vector"/>
 </instance>
 <instance part="P+9" gate="G$1" x="322.58" y="144.78" smashed="yes">
@@
 </segment>
 <segment>
-<pinref part="R4" gate="G$1" pin="2"/>
-<pinref part="P+10" gate="G$1" pin="3.3V"/>
-<wire x1="337.82" y1="142.24" x2="337.82" y2="144.78" width="0.1524" layer="91"/>
-</segment>
-<segment>
 <wire x1="91.44" y1="83.82" x2="91.44" y2="86.36" width="0.1524" layer="91"/>
 <wire x1="99.06" y1="83.82" x2="99.06" y2="86.36" width="0.1524" layer="91"/>
@@
 <junction x="195.58" y="121.92"/>
 <pinref part="U4" gate="G$1" pin="VDD"/>
+</segment>
+<segment>
+<pinref part="LED3" gate="G$1" pin="A"/>
+<pinref part="P+10" gate="G$1" pin="3.3V"/>
+<wire x1="337.82" y1="139.7" x2="337.82" y2="144.78" width="0.1524" layer="91"/>
 </segment>
 </net>
@@
 </segment>
 </net>
-<net name="N$9" class="0">
-<segment>
-<pinref part="U6" gate="G$1" pin="P0_2"/>
-<pinref part="LED3" gate="G$1" pin="C"/>
-<wire x1="320.04" y1="129.54" x2="327.66" y2="129.54" width="0.1524" layer="91"/>
-</segment>
-</net>
-<net name="N$10" class="0">
-<segment>
-<pinref part="LED3" gate="G$1" pin="A"/>
-<pinref part="R4" gate="G$1" pin="1"/>
-<wire x1="335.28" y1="129.54" x2="337.82" y2="129.54" width="0.1524" layer="91"/>
-<wire x1="337.82" y1="129.54" x2="337.82" y2="132.08" width="0.1524" layer="91"/>
-</segment>
-</net>
 <net name="BT_RX" class="0">
 <segment>
@@
 </segment>
 </net>
+<net name="N$1" class="0">
+<segment>
+<pinref part="U6" gate="G$1" pin="P0_2"/>
+<pinref part="R4" gate="G$1" pin="2"/>
+<wire x1="320.04" y1="129.54" x2="325.12" y2="129.54" width="0.1524" layer="91"/>
+</segment>
+</net>
+<net name="N$5" class="0">
+<segment>
+<pinref part="R4" gate="G$1" pin="1"/>
+<pinref part="LED3" gate="G$1" pin="C"/>
+<wire x1="335.28" y1="129.54" x2="337.82" y2="129.54" width="0.1524" layer="91"/>
+<wire x1="337.82" y1="129.54" x2="337.82" y2="132.08" width="0.1524" layer="91"/>
+</segment>
+</net>

Commit message: Version 1.1 complete and ready for fab.
Parts:
- R2, R3: value 333 -> 100
Other:
- note added: "v1.1 Nov 29, 2017 Fixed switch footprint Moved BLE led to edge of board 2-pin power screw terminal now 3.5mm PRG and RESET lables corrected LED resistors changed to 8K to dim the LEDs Added pin numbers to output header silk Switched reset controller to SOT-23 (SC70 not available)"
Changed lines of the file:
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@@
 <part name="GND21" library="SparkFun-Aesthetics" deviceset="GND" device=""/>
 <part name="U$5" library="SchmalzHaus" deviceset="SCHMALZHAUS" device="SCHMALZHAUS_SMALL"/>
-<part name="R2" library="SparkFun-Resistors" deviceset="RESISTOR" device="0603" value="333"/>
-<part name="R3" library="SparkFun-Resistors" deviceset="RESISTOR" device="0603" value="333"/>
+<part name="R2" library="SparkFun-Resistors" deviceset="RESISTOR" device="0603" value="100"/>
+<part name="R3" library="SparkFun-Resistors" deviceset="RESISTOR" device="0603" value="100"/>
 <part name="C11" library="SparkFun-Capacitors" deviceset="CAP_POL" device="C" value="100uF"/>
 <part name="GND25" library="SparkFun-Aesthetics" deviceset="GND" device=""/>
@@
 <text x="204.216" y="182.372" size="1.27" layer="98" font="vector">5V</text>
 <text x="204.216" y="179.832" size="1.27" layer="98" font="vector">GND</text>
-<text x="7.62" y="223.012" size="1.778" layer="98">v1.0 Nov 9, 2017
+<text x="7.62" y="223.012" size="1.4224" layer="98">v1.0 Nov 9, 2017
    Initial release</text>
-<text x="7.62" y="228.6" size="1.778" layer="98">Version History</text>
+<text x="7.62" y="228.6" size="1.4224" layer="98">Version History</text>
 <text x="227.838" y="176.022" size="1.27" layer="98" font="vector" rot="R180">GND</text>
 <text x="7.62" y="241.3" size="2.54" layer="98" ratio="15">A DIP form factor chipKIT® compatible board</text>
@@
 <text x="204.47" y="71.628" size="1.27" layer="98" font="vector">Power and Pin 1 LEDs</text>
 <text x="308.864" y="96.52" size="1.27" layer="98" font="vector">PRG and RST Buttons</text>
+<text x="7.62" y="205.232" size="1.4224" layer="98">v1.1 Nov 29, 2017
+   Fixed switch footprint
+   Moved BLE led to edge of board
+   2-pin power screw terminal now 3.5mm
+   PRG and RESET lables corrected
+   LED resistors changed to 8K to dim the LEDs
+   Added pin numbers to output header silk
+   Switched reset controller to SOT-23 (SC70 not available)</text>
 </plain>
 <instances>
