File: board_v12/RGB_Station_v12.sch (EAGLE design)
At the start: 44 parts, among them IC1 MCP1702T-3302E/MB, J1 M20, J2 M20, J3 USB_MICRO, SW1 KMR2_SWITCH, SW2 KMR2_SWITCH, U1 PIC32MX270F256D_44VTLA_44, U2 74LVC2T45, U3 MCP131T-315E/TT, U4 DSC6111CI1A-008.0000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

Commit message: Done with pin diagram.
Other:
- note added: "Both DotStar and NeoPixels can be used with this board. NeoPixe (WS2812): Use +5V, GND, and DAT pins on connector. In code, use output pin 18. DotStar (APA102): Use +5V, GND, DAT and CLK pins In code, use defualt SPI port"
- note removed: "Both DotStar and NeoPixels can be used with this board. NeoPixel: Use +5V, GND, and DAT pins on connector. In code, use output pin 18. DotStar: Use +5V, GND, DAT and CLK pins In code, use defualt SPI port"
Changed lines of the file:
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@@
 <text x="331.724" y="205.994" size="1.27" layer="98" font="vector">Both DotStar and NeoPixels can
 be used with this board.
-NeoPixel:
+NeoPixe (WS2812):
   Use +5V, GND, and DAT pins
   on connector. In code, use
   output pin 18.
-DotStar:
+DotStar (APA102):
   Use +5V, GND, DAT and CLK pins
   In code, use defualt SPI port
